File: keyboard-project.kicad_sch (KiCad schematic)
At the start: 0 parts

Commit message: Schematic editing
Parts:
- added C1: 1uF, symbol Device:C_Small
- added R1: 10k, symbol Device:R_Small
- added R2, R3: 22, symbol Device:R_Small
- added U1: ATmega32U4-A, Package_QFP:TQFP-44_10x10mm_P0.8mm, symbol MCU_Microchip_ATmega:ATmega32U4-A
Connections:
- new net: R3.2, U1.3 (D-)
- new net: C1.1, U1.6 (UCAP)
- new net: R1.1, U1.33 (~{HWB}/PE2)
- new net: R2.2, U1.4 (D+)
- new net +5V: U1.14 (VCC), U1.2 (UVCC), U1.24 (AVCC), U1.34 (VCC), U1.44 (AVCC)
- new net GND: C1.2, R1.2, U1.15 (GND), U1.23 (GND), U1.35 (GND), U1.43 (GND), U1.5 (UGND)
